File: matrix.sch (KiCad schematic (older format))
At the start: 134 parts, among them K0:0 KEYSW, K0:1 KEYSW, K0:2 KEYSW, K0:3 KEYSW, K0:4 KEYSW, K10:0 KEYSW, K10:1 KEYSW, K10:2 KEYSW, K10:3 KEYSW, K10:4 KEYSW, K11:0 KEYSW, K11:1 KEYSW, K11:2 KEYSW, K11:3 KEYSW, K11:4 KEYSW, K12:0 KEYSW, K12:1 KEYSW, K12:2 KEYSW, K12:3 KEYSW, K12:4 KEYSW, K13:0 KEYSW, K13:1 KEYSW, K13:2 KEYSW, K13:3 KEYSW, K13:4 KEYSW, K1:0 KEYSW, K1:1 KEYSW, K1:2 KEYSW, K1:3 KEYSW, K1:4 KEYSW, K2:0 KEYSW, K2:1 KEYSW, K2:2 KEYSW, K2:3 KEYSW, K2:4 KEYSW, K3:0 KEYSW, K3:1 KEYSW, K3:2 KEYSW, K3:3 KEYSW, K3:4 KEYSW, K4:0 KEYSW, K4:1 KEYSW, K4:2 KEYSW, K4:3 KEYSW, K4:4 KEYSW, K5:0 KEYSW, K5:1 KEYSW, K5:2 KEYSW, K5:3 KEYSW, K5:4 KEYSW, K6:0 KEYSW, K6:1 KEYSW, K6:3 KEYSW, K7:0 KEYSW, K7:1 KEYSW, K7:3 KEYSW, K7:4 KEYSW, K8:0 KEYSW, K8:1 KEYSW, K8:2 KEYSW, K8:3 KEYSW, K8:4 KEYSW, K9:0 KEYSW, K9:1 KEYSW, K9:2 KEYSW, K9:3 KEYSW, K9:4 KEYSW

Commit message: Temp #2
Parts:
- D6:1, D6:3, D7:1, D7:3: footprint keyboard_parts:Mx_Alps_150_VERT -> keyboard_parts:D_SOD123_axial
Changed lines of the file:
@@
 F 0 "D6:1" V 4800 3400 60  0000 C CNN
 F 1 "D" V 5100 3400 60  0001 C CNN
-F 2 "keyboard_parts:Mx_Alps_150_VERT" H 4950 3450 60  0001 C CNN
+F 2 "keyboard_parts:D_SOD123_axial" H 4950 3450 60  0001 C CNN
 F 3 "" H 4950 3450 60  0000 C CNN
 	1    4950 3450
@@
 F 0 "D6:3" V 4800 4700 60  0000 C CNN
 F 1 "D" V 5100 4700 60  0001 C CNN
-F 2 "keyboard_parts:Mx_Alps_150_VERT" H 4950 4750 60  0001 C CNN
+F 2 "keyboard_parts:D_SOD123_axial" H 4950 4750 60  0001 C CNN
 F 3 "" H 4950 4750 60  0000 C CNN
 	1    4950 4750
@@
 F 0 "D7:1" V 5850 3400 60  0000 C CNN
 F 1 "D" V 6150 3400 60  0001 C CNN
-F 2 "keyboard_parts:Mx_Alps_150_VERT" H 6000 3450 60  0001 C CNN
+F 2 "keyboard_parts:D_SOD123_axial" H 6000 3450 60  0001 C CNN
 F 3 "" H 6000 3450 60  0000 C CNN
 	1    6000 3450
@@
 F 0 "D7:3" V 5850 4700 60  0000 C CNN
 F 1 "D" V 6150 4700 60  0001 C CNN
-F 2 "keyboard_parts:Mx_Alps_150_VERT" H 6000 4750 60  0001 C CNN
+F 2 "keyboard_parts:D_SOD123_axial" H 6000 4750 60  0001 C CNN
 F 3 "" H 6000 4750 60  0000 C CNN
 	1    6000 4750
