File: ergowing-pcb.kicad_pcb (KiCad board)
At the start: 2 copper layers, 150 parts, among them J1 USB_mini_micro_B, K0:0 KEYSW, K0:1 KEYSW, K0:2 KEYSW, K0:3 KEYSW, K0:4 KEYSW, K10:0 KEYSW, K10:1 KEYSW, K10:2 KEYSW, K10:3 KEYSW, K10:4 KEYSW, K11:0 KEYSW, K11:1 KEYSW, K11:2 KEYSW, K11:3 KEYSW, K11:4 KEYSW, K12:0 KEYSW, K12:1 KEYSW, K12:2 KEYSW, K12:3 KEYSW, K12:4 KEYSW, K13:0 KEYSW, K13:1 KEYSW, K13:2 KEYSW, K13:3 KEYSW, K13:4 KEYSW, K1:0 KEYSW, K1:1 KEYSW, K1:2 KEYSW, K1:3 KEYSW, K1:4 KEYSW, K2:0 KEYSW, K2:1 KEYSW, K2:2 KEYSW, K2:3 KEYSW, K2:4 KEYSW, K3:0 KEYSW, K3:1 KEYSW, K3:2 KEYSW, K3:3 KEYSW, K3:4 KEYSW, K4:0 KEYSW, K4:1 KEYSW, K4:2 KEYSW, K4:3 KEYSW, K4:4 KEYSW, K5:0 KEYSW, K5:1 KEYSW, K5:2 KEYSW, K5:3 KEYSW, K5:4 KEYSW, K6:0 KEYSW, K6:1 KEYSW, K6:3 KEYSW, K7:0 KEYSW, K7:1 KEYSW, K7:3 KEYSW, K7:4 KEYSW, K8:0 KEYSW, K8:1 KEYSW, K8:2 KEYSW, K8:3 KEYSW, K8:4 KEYSW, K9:0 KEYSW, K9:1 KEYSW, K9:2 KEYSW, K9:3 KEYSW, K9:4 KEYSW, SW1 SW_PUSH, U1 ATMEGA32U4, X1 XTAL_GND

Commit message: Place components
Parts:
- moved J1 225.9 mm to (198.9, 45.9)
- moved C1 185.7 mm to (194.2, 100.7), turned to 90 degrees
- moved C2 185.1 mm to (203.1, 100.7), turned to 90 degrees
- moved C6 183.3 mm to (189.4, 100.7), turned to 90 degrees
- moved C4 181.5 mm to (208.5, 107.8), turned to 270 degrees
- moved C8 178.9 mm to (189.4, 112.6), turned to 90 degrees
- moved C5 174.0 mm to (189.4, 107.8), turned to 90 degrees
- moved R4 173.4 mm to (197.7, 95.9)
- moved R3 173.1 mm to (191.2, 95.9)
- moved C7 171.4 mm to (189.4, 117.4), turned to 90 degrees
- moved C3 170.0 mm to (208.5, 117.4), turned to 270 degrees
- moved X1 168.4 mm to (198.9, 100.7), turned to 45 degrees
- moved U1 164.2 mm to (198.9, 112.6)
- moved R2 158.1 mm to (208.5, 112.6), turned to 90 degrees
- moved SW1 145.5 mm to (198.9, 125.7)
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
Commit message: Edge cut defined?
Parts:
- added K0:0: KEYSW, keebs:Mx_Alps_150_R-5deg, F.Cu at (-15.2, 41.8)
Other:
- board outline added: 388.1 x 110.8 mm
Changed lines of the file:
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@@
 (kicad_pcb (version 4) (host pcbnew 4.0.7)
   (general
-    (links 515)
-    (no_connects 247)
-    (area 43.748094 28.857392 354.051906 279.9875)
+    (links 517)
+    (no_connects 249)
+    (area -29.596701 20.324999 361.109533 137.475001)
     (thickness 1.6)
-    (drawings 0)
+    (drawings 22)
     (tracks 0)
     (zones 0)
-    (modules 150)
+    (modules 151)
     (nets 107)
   )
@@
     (38 B.Mask user)
     (39 F.Mask user)
-    (40 Dwgs.User user)
+    (40 Dwgs.User user hide)
     (41 Cmts.User user)
     (42 Eco1.User user)
@@
     (add_net row4)
   )
+  (module keebs:Mx_Alps_150_R-5deg (layer F.Cu)
+    (at -15.16 41.83 5)
+    (descr MXALPS)
+    (tags MXALPS)
+    (fp_text reference K0:0 (at 0.386308 -2.551039 360) (layer B.SilkS)
+      (effects (font (size 1 1) (thickness 0.2)) (justify mirror))
+    )
+    (fp_text value KEYSW (at 8.91639 11.743803 360) (layer B.SilkS) hide
+      (effects (font (thickness 0.3048)) (justify mirror))
+    )
+    (fp_line (start -5.772397 -6.879275) (end 6.879275 -5.772397) (layer Cmts.User) (width 0.1524))
+    (fp_line (start 6.879275 -5.772397) (end 5.772397 6.879275) (layer Cmts.User) (width 0.1524))
+    (fp_line (start 5.772397 6.879275) (end -6.879275 5.772397) (layer Cmts.User) (width 0.1524))
+    (fp_line (start -6.879275 5.772397) (end -5.772397 -6.879275) (layer Cmts.User) (width 0.1524))
+    (fp_line (start -13.287525 -10.596407) (end 14.925705 -8.128069) (layer Dwgs.User) (width 0.1524))
+    (fp_line (start 14.925705 -8.128069) (end 13.287525 10.596407) (layer Dwgs.User) (width 0.1524))
+    (fp_line (start 13.287525 10.596407) (end -14.925705 8.128069) (layer Dwgs.User) (width 0.1524))
+    (fp_line (start -14.925705 8.128069) (end -13.287525 -10.596407) (layer Dwgs.User) (width 0.1524))
+    (fp_line (start -5.772397 -6.879275) (end -4.001163 -6.724312) (layer F.SilkS) (width 0.381))
+    (fp_line (start 5.108041 -5.92736) (end 6.879275 -5.772397) (layer F.SilkS) (width 0.381))
+    (fp_line (start 6.879275 -5.772397) (end 6.724312 -4.001163) (layer F.SilkS) (width 0.381))
+    (fp_line (start 5.92736 5.108041) (end 5.772397 6.879275) (layer F.SilkS) (width 0.381))
+    (fp_line (start 5.772397 6.879275) (end 4.001163 6.724312) (layer F.SilkS) (width 0.381))
+    (fp_line (start -5.108041 5.92736) (end -6.879275 5.772397) (layer F.SilkS) (width 0.381))
+    (fp_line (start -6.879275 5.772397) (end -6.724312 4.001163) (layer F.SilkS) (width 0.381))
+    (fp_line (start -5.92736 -5.108041) (end -5.772397 -6.879275) (layer F.SilkS) (width 0.381))
+    (fp_line (start -6.349637 -7.567203) (end 7.567203 -6.349637) (layer Eco2.User) (width 0.1524))
+    (fp_line (start 7.567203 -6.349637) (end 6.349637 7.567203) (layer Eco2.User) (width 0.1524))
+    (fp_line (start 6.349637 7.567203) (end -7.567203 6.349637) (layer Eco2.User) (width 0.1524))
+    (fp_line (start -7.567203 6.349637) (end -6.349637 -7.567203) (layer Eco2.User) (width 0.1524))
+    (fp_line (start -8.278306 5.700189) (end -7.162712 -7.051103) (layer Dwgs.User) (width 0.3))
+    (fp_line (start -8.278306 5.700189) (end 7.162712 7.051103) (layer Dwgs.User) (width 0.3))
+    (fp_line (start 7.162712 7.051103) (end 8.278306 -5.700189) (layer Dwgs.User) (width 0.3))
+    (fp_line (start 8.278306 -5.700189) (end -7.162712 -7.051103) (layer Dwgs.User) (width 0.3))
+    (fp_line (start -6.926877 -8.25513) (end 8.25513 -6.926877) (layer Dwgs.User) (width 0.3))
+    (fp_line (start 8.25513 -6.926877) (end 6.926877 8.25513) (layer Dwgs.User) (width 0.3))
+    (fp_line (start 6.926877 8.25513) (end -8.25513 6.926877) (layer Dwgs.User) (width 0.3))
+    (fp_line (start -8.25513 6.926877) (end -6.926877 -8.25513) (layer Dwgs.User) (width 0.3))
+    (pad HOLE np_thru_hole circle (at 0 0) (size 3.9878 3.9878) (drill 3.9878) (layers *.Cu))
+    (pad HOLE np_thru_hole circle (at -5.060669 -0.442751) (size 1.7018 1.7018) (drill 1.7018) (layers *.Cu))
+    (pad HOLE np_thru_hole circle (at 5.060669 0.442751) (size 1.7018 1.7018) (drill 1.7018) (layers *.Cu))
+    (pad 1 thru_hole oval (at -3.107044 -3.554322 330.95) (size 2.5 4.17) (drill oval 1.5 3.17) (layers *.Cu *.Mask F.SilkS)
+      (net 81 col0))
+    (pad 2 thru_hole oval (at 2.927887 -4.55214 356.1) (size 2.5 3.08) (drill oval 1.5 2.08) (layers *.Cu *.Mask F.SilkS)
+      (net 6 "Net-(D0:0-Pad2)"))
+  )
   (module Capacitors_SMD:C_0805_HandSoldering (layer B.Cu)
     (at 194.165625 100.701563 90)
@@
       (net 77 "Net-(D13:4-Pad2)"))
   )
+  (gr_line (start 213 135.2) (end 352.44 123) (angle 90) (layer Edge.Cuts) (width 0.15))
+  (gr_line (start 345.3 25.67) (end 353.68 121.48) (angle 90) (layer Edge.Cuts) (width 0.15))
+  (gr_line (start 204.85 36.54) (end 343.78 24.39) (angle 90) (layer Edge.Cuts) (width 0.15))
+  (gr_arc (start 343.91 25.78) (end 343.787982 24.385327) (angle 90) (layer Edge.Cuts) (width 0.15))
+  (gr_arc (start 352.29 121.61) (end 353.684673 121.487982) (angle 90) (layer Edge.Cuts) (width 0.15))
+  (gr_line (start 185 135.2) (end 45.4 122.87) (angle 90) (layer Edge.Cuts) (width 0.15))
+  (gr_line (start 192.95 36.54) (end 54.02 24.41) (angle 90) (layer Edge.Cuts) (width 0.15))
+  (gr_line (start 52.51 25.68) (end 44.12 121.48) (angle 90) (layer Edge.Cuts) (width 0.15))
+  (gr_arc (start 45.525 121.48) (end 45.402982 122.874673) (angle 90) (layer Edge.Cuts) (width 0.15))
+  (gr_arc (start 53.9 25.8) (end 52.505327 25.677982) (angle 90) (layer Edge.Cuts) (width 0.15))
+  (gr_arc (start -32.98 34.46) (end -32.98 35.86) (angle 90) (layer Edge.Cuts) (width 0.15))
+  (gr_line (start -29.4 49.9) (end -29.4 33.7) (angle 90) (layer Edge.Cuts) (width 0.15))
+  (gr_line (start -2.3 51.3) (end -28 51.3) (angle 90) (layer Edge.Cuts) (width 0.15))
+  (gr_line (start -0.9 33.7) (end -0.9 49.9) (angle 90) (layer Edge.Cuts) (width 0.15))
+  (gr_line (start -28 32.3) (end -2.3 32.3) (angle 90) (layer Edge.Cuts) (width 0.15))
+  (gr_arc (start -2.3 33.7) (end -2.3 32.3) (angle 90) (layer Edge.Cuts) (width 0.15))
+  (gr_arc (start -2.3 49.9) (end -0.9 49.9) (angle 90) (layer Edge.Cuts) (width 0.15))
+  (gr_arc (start -28 49.9) (end -28 51.3) (angle 90) (layer Edge.Cuts) (width 0.15))
+  (gr_arc (start -32 32.1) (end -32 33.5) (angle 90) (layer Edge.Cuts) (width 0.15))
+  (gr_arc (start -28 33.7) (end -29.4 33.7) (angle 90) (layer Edge.Cuts) (width 0.15))
+  (gr_line (start 192.95 36.54) (end 204.85 36.54) (angle 90) (layer Edge.Cuts) (width 0.15))
+  (gr_line (start 185 135.2) (end 213 135.2) (angle 90) (layer Edge.Cuts) (width 0.15))
 )

Commit message: Zones complete
Parts:
- moved J1 3.57 mm to (198.9, 42.4)
Routing:
- added copper zone on B.Cu, net GND
- added copper zone on F.Cu, net GND
Changed lines of the file:
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@@
   (general
     (links 517)
-    (no_connects 249)
-    (area -29.596701 20.324999 361.109533 137.475001)
+    (no_connects 235)
+    (area -34.455001 24.304999 354.051906 135.97534)
     (thickness 1.6)
     (drawings 22)
@@
     (38 B.Mask user)
     (39 F.Mask user)
-    (40 Dwgs.User user hide)
+    (40 Dwgs.User user)
     (41 Cmts.User user)
     (42 Eco1.User user)
@@
   )
   (module keyboard_parts:USB_miniB_hirose_5S8 (layer B.Cu)
-    (at 198.928125 45.932813)
+    (at 198.928125 42.360938)
     (descr "USB miniB hirose UX60SC-MB-5S8")
     (tags "USB miniB hirose through hole UX60SC-MB-5S8")
@@
   (gr_line (start 192.95 36.54) (end 204.85 36.54) (angle 90) (layer Edge.Cuts) (width 0.15))
   (gr_line (start 185 135.2) (end 213 135.2) (angle 90) (layer Edge.Cuts) (width 0.15))
+  (zone (net 2) (net_name GND) (layer F.Cu) (hatch edge 0.508)
+    (connect_pads (clearance 0.508))
+    (min_thickness 0.254)
+    (fill yes (arc_segments 16) (thermal_gap 0.508) (thermal_bridge_width 0.508))
+    (polygon
+      (pts
+        (xy 44.05 122.71) (xy 52.64 24.29) (xy 192.9 36.54) (xy 204.95 36.53) (xy 345.19 24.28)
+        (xy 353.77 122.82) (xy 213.02 135.22) (xy 184.92 135.19) (xy 44.06 122.71)
+      )
+    )
+  )
+  (zone (net 2) (net_name GND) (layer B.Cu) (hatch edge 0.508)
+    (connect_pads (clearance 0.508))
+    (min_thickness 0.254)
+    (fill yes (arc_segments 16) (thermal_gap 0.508) (thermal_bridge_width 0.508))
+    (polygon
+      (pts
+        (xy 44.05 122.71) (xy 52.64 24.29) (xy 192.9 36.54) (xy 204.95 36.53) (xy 345.19 24.28)
+        (xy 353.77 122.82) (xy 213.02 135.22) (xy 184.92 135.19) (xy 44.06 122.71)
+      )
+    )
+  )
 )

Commit message: Pre-switch wiring
Parts:
- removed the K0:0 at (-15.2, 41.8)
Routing:
- net VCC: track 0.00 -> 156.1 mm
- net Net-(J1-Pad2): track 0.00 -> 57.0 mm
- net Net-(J1-Pad3): track 0.00 -> 54.6 mm
- net GND: track 0.00 -> 36.4 mm, vias 0 -> 6
- net Net-(R1-Pad2): track 0.00 -> 33.5 mm, vias 0 -> 2
- net Net-(R4-Pad2): track 0.00 -> 25.3 mm, vias 0 -> 2
- net Net-(R3-Pad2): track 0.00 -> 21.4 mm, vias 0 -> 2
- net Net-(C1-Pad1): track 0.00 -> 10.7 mm
- net Net-(C2-Pad1): track 0.00 -> 10.4 mm
- net Net-(R2-Pad1): track 0.00 -> 4.92 mm
- net Net-(C8-Pad1): track 0.00 -> 4.34 mm
Other:
- board size 388.1 x 110.8 mm -> 309.6 x 110.8 mm

Commit message: Revert "Revert "Rows wired""
This reverts commit adba6586d6cb1fc90ef0a2f50d1a669c9e1cd072.
Routing:
- net Net-(K5:0-Pad1): track 0.00 -> 109.4 mm
- net col7: track 0.00 -> 108.9 mm
- net col8: track 0.00 -> 100.5 mm
- net col1: track 0.00 -> 100.0 mm
- net col2: track 0.00 -> 99.4 mm
- net col10: track 0.00 -> 99.3 mm
- net col13: track 0.00 -> 99.1 mm
- net col4: track 0.00 -> 99.0 mm
- net col3: track 0.00 -> 98.2 mm
- net col12: track 0.00 -> 98.1 mm
- net col0: track 0.00 -> 97.9 mm
- net col9: track 0.00 -> 84.5 mm
- net col11: track 0.00 -> 84.3 mm
- net col6: track 0.00 -> 79.2 mm

Commit message: Connect switches to diodes
Parts:
- moved D7:3 6.35 mm to (220.1, 103.9), turned to 5 degrees
- moved D6:1 6.23 mm to (180.4, 75.9), turned to 355 degrees
- moved D6:3 6.23 mm to (177.9, 103.9), turned to 355 degrees
- moved D7:1 6.20 mm to (217.6, 76.0), turned to 5 degrees
- turned K6:1 to 355 degrees
- turned K6:3 to 355 degrees
- turned K7:1 to 5 degrees
- turned K7:3 to 5 degrees
Routing:
- net col7: track 108.9 -> 93.7 mm
- net col9: track 84.5 -> 99.0 mm
- net col6: track 79.2 -> 66.8 mm
- net Net-(D10:1-Pad2): track 0.00 -> 9.97 mm
- net Net-(D13:2-Pad2): track 0.00 -> 9.92 mm
- net Net-(D13:0-Pad2): track 0.00 -> 9.92 mm
- net Net-(D10:2-Pad2): track 0.00 -> 9.91 mm
- net Net-(D12:2-Pad2): track 0.00 -> 9.90 mm
- net Net-(D7:4-Pad2): track 0.00 -> 9.90 mm
- net Net-(D11:1-Pad2): track 0.00 -> 9.89 mm
- net Net-(D6:1-Pad2): track 0.00 -> 9.89 mm
- net Net-(D8:1-Pad2): track 0.00 -> 9.89 mm
- net Net-(D13:3-Pad2): track 0.00 -> 9.89 mm
- net Net-(D7:3-Pad2): track 0.00 -> 9.89 mm
- net Net-(D10:3-Pad2): track 0.00 -> 9.88 mm
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
Commit message: Revert "Connect switches to diodes"
This reverts commit 2486d4e9eff35fc84fffcee9a461cbe5a4c6410b.
Parts:
- moved D7:3 6.35 mm to (215.2, 99.8), turned to 275 degrees
- moved D6:1 6.23 mm to (176.3, 71.2), turned to 265 degrees
- moved D6:3 6.23 mm to (173.8, 99.2), turned to 265 degrees
- moved D7:1 6.20 mm to (212.8, 72.1), turned to 275 degrees
- turned K6:1 to 265 degrees
- turned K6:3 to 265 degrees
- turned K7:1 to 275 degrees
- turned K7:3 to 275 degrees
Routing:
- net col7: track 93.7 -> 108.9 mm
- net col9: track 99.0 -> 84.5 mm
- net col6: track 66.8 -> 79.2 mm
- net Net-(D10:1-Pad2): track 9.97 -> 0.00 mm
- net Net-(D13:2-Pad2): track 9.92 -> 0.00 mm
- net Net-(D13:0-Pad2): track 9.92 -> 0.00 mm
- net Net-(D10:2-Pad2): track 9.91 -> 0.00 mm
- net Net-(D12:2-Pad2): track 9.90 -> 0.00 mm
- net Net-(D7:4-Pad2): track 9.90 -> 0.00 mm
- net Net-(D11:1-Pad2): track 9.89 -> 0.00 mm
- net Net-(D6:1-Pad2): track 9.89 -> 0.00 mm
- net Net-(D8:1-Pad2): track 9.89 -> 0.00 mm
- net Net-(D13:3-Pad2): track 9.89 -> 0.00 mm
- net Net-(D7:3-Pad2): track 9.89 -> 0.00 mm
- net Net-(D10:3-Pad2): track 9.88 -> 0.00 mm
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
Commit message: Revert "Rows wired"
This reverts commit d70f662c53e392adef38fe5ef701a55c1d48fb42.
Routing:
- net Net-(K5:0-Pad1): track 109.4 -> 0.00 mm
- net col7: track 108.9 -> 0.00 mm
- net col8: track 100.5 -> 0.00 mm
- net col1: track 100.0 -> 0.00 mm
- net col2: track 99.4 -> 0.00 mm
- net col10: track 99.3 -> 0.00 mm
- net col13: track 99.1 -> 0.00 mm
- net col4: track 99.0 -> 0.00 mm
- net col3: track 98.2 -> 0.00 mm
- net col12: track 98.1 -> 0.00 mm
- net col0: track 97.9 -> 0.00 mm
- net col9: track 84.5 -> 0.00 mm
- net col11: track 84.3 -> 0.00 mm
- net col6: track 79.2 -> 0.00 mm
